File: embedded/Schemes/First_schemes/First_schemes.kicad_sch (KiCad schematic)
At the start: 5 parts

Commit message: More trusted scheme
Parts:
- added C1, C4: 100uF, symbol Device:C_Polarized_US
- added C2, C3: 0.1uF, symbol Device:C
- added M1: Servo, symbol Motor:Motor_Servo
- added U6: LM7805_TO220, Package_TO_SOT_THT:TO-220-3_Vertical, symbol Regulator_Linear:LM7805_TO220
Connections:
- net +5V: now also C3.1, C4.1, U6.3 (VO)
- net GND: now also C1.2, C2.2, C3.2, C4.2, M1.3 (-), U6.2 (GND)
- net at U5.28 (GPIO42): now also M1.1 (PWM)
- net at U5.29 (GPIO41): now also M1.2 (+)
- new net +12V: C1.1, C2.1, U6.1 (VI)

Commit message: Trustworthy schematic
Parts:
- removed C1, C4: 100uF, symbol Device:C_Polarized_US
- removed C2, C3: 0.1uF, symbol Device:C
- removed M1: Servo, symbol Motor:Motor_Servo
- removed U6: LM7805_TO220, Package_TO_SOT_THT:TO-220-3_Vertical, symbol Regulator_Linear:LM7805_TO220
- added J1: Barrel_Jack, symbol Connector:Barrel_Jack
- added M1: Motor, symbol Motor:Motor_DC
- added U6: Relay, symbol Symbols:Relay
Connections:
- net +5V: now also U6.1 (VCC)
- net GND: now also J1.2, M1.2 (-), U6.2 (GND)
- net at U5.30 (GPIO40): now also U6.3 (In1)
- new net: M1.1 (+), U6.4 (NO)
- new net: J1.1, U6.5 (C)

Commit message: The trustiest scheme
Connections:
- net +5V: now also J1.1, U6.5 (C)
- net at U5.30 (GPIO40): no longer U6.3 (In1)
- net SCL: now reaches U5.4 (GPIO4)
- net SCL: now also U4.4 (SCL)
- net at U5.40 (GPIO21): no longer U4.3 (SDA)
- net at U5.41 (GPIO20): no longer U4.4 (SCL)
- net SDA: now reaches U5.5 (GPIO5)
- net SDA: now also U4.3 (SDA)
- net Motor: now reaches U5.6 (GPIO6)
- net Motor: now also U6.3 (In1)
- net IR: now reaches U5.7 (GPIO7)
- net IR: now also U2.3 (In)
- removed net IR_sensor: U2.3 (In), U5.42 (GPIO19)
Other:
- note added: "Изготвено от: A4 само хартия"
- moved on the sheet: M1
Changed lines of the file:
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@@
 (kicad_sch (version 20230121) (generator eeschema)
   (paper "A4")
-  (wire (pts (xy 64.77 33.02) (xy 64.77 34.29))
+  (junction (at 132.08 31.75) (diameter 0) (color 0 0 0 0)
+  )
+  (wire (pts (xy 54.61 33.02) (xy 54.61 27.94))
     (stroke (width 0) (type default))
   )
@@
     (stroke (width 0) (type default))
   )
-  (wire (pts (xy 95.25 67.31) (xy 110.49 67.31))
-    (stroke (width 0) (type default))
-  )
   (wire (pts (xy 40.64 30.48) (xy 40.64 25.4))
     (stroke (width 0) (type default))
@@
     (stroke (width 0) (type default))
   )
-  (wire (pts (xy 95.25 39.37) (xy 106.68 39.37))
-    (stroke (width 0) (type default))
-  )
-  (wire (pts (xy 114.3 64.77) (xy 114.3 104.14))
-    (stroke (width 0) (type default))
-  )
   (wire (pts (xy 50.8 105.41) (xy 49.53 105.41))
     (stroke (width 0) (type default))
@@
     (stroke (width 0) (type default))
   )
+  (wire (pts (xy 132.08 31.75) (xy 132.08 36.83))
+    (stroke (width 0) (type default))
+  )
   (wire (pts (xy 39.37 38.1) (xy 59.69 38.1))
     (stroke (width 0) (type default))
@@
     (stroke (width 0) (type default))
   )
+  (wire (pts (xy 97.79 39.37) (xy 106.68 39.37))
+    (stroke (width 0) (type default))
+  )
   (wire (pts (xy 50.8 118.11) (xy 49.53 118.11))
     (stroke (width 0) (type default))
@@
     (stroke (width 0) (type default))
   )
-  (wire (pts (xy 39.37 33.02) (xy 64.77 33.02))
+  (wire (pts (xy 39.37 33.02) (xy 54.61 33.02))
     (stroke (width 0) (type default))
   )
@@
     (stroke (width 0) (type default))
   )
-  (wire (pts (xy 127 34.29) (xy 127 40.64))
+  (wire (pts (xy 127 34.29) (xy 127 38.1))
     (stroke (width 0) (type default))
   )
@@
     (stroke (width 0) (type default))
   )
+  (wire (pts (xy 125.73 31.75) (xy 132.08 31.75))
+    (stroke (width 0) (type default))
+  )
   (wire (pts (xy 50.8 97.79) (xy 49.53 97.79))
     (stroke (width 0) (type default))
@@
     (stroke (width 0) (type default))
   )
+  (wire (pts (xy 63.5 34.29) (xy 68.58 34.29))
+    (stroke (width 0) (type default))
+  )
   (wire (pts (xy 53.34 19.05) (xy 53.34 21.59))
     (stroke (width 0) (type default))
@@
     (stroke (width 0) (type default))
   )
+  (wire (pts (xy 57.15 27.94) (xy 57.15 30.48))
+    (stroke (width 0) (type default))
+  )
   (wire (pts (xy 44.45 69.85) (xy 68.58 69.85))
     (stroke (width 0) (type default))
@@
     (stroke (width 0) (type default))
   )
-  (wire (pts (xy 114.3 104.14) (xy 80.01 104.14))
-    (stroke (width 0) (type default))
-  )
-  (wire (pts (xy 110.49 67.31) (xy 110.49 106.68))
+  (wire (pts (xy 63.5 31.75) (xy 68.58 31.75))
     (stroke (width 0) (type default))
   )
@@
     (stroke (width 0) (type default))
   )
+  (wire (pts (xy 54.61 27.94) (xy 57.15 27.94))
+    (stroke (width 0) (type default))
+  )
   (wire (pts (xy 50.8 87.63) (xy 49.53 87.63))
     (stroke (width 0) (type default))
@@
     (stroke (width 0) (type default))
   )
-  (wire (pts (xy 132.08 29.21) (xy 132.08 36.83))
+  (wire (pts (xy 132.08 29.21) (xy 132.08 31.75))
     (stroke (width 0) (type default))
   )
@@
     (stroke (width 0) (type default))
   )
+  (wire (pts (xy 63.5 29.21) (xy 68.58 29.21))
+    (stroke (width 0) (type default))
+  )
   (wire (pts (xy 41.91 69.85) (xy 41.91 73.66))
     (stroke (width 0) (type default))
@@
     (stroke (width 0) (type default))
   )
-  (wire (pts (xy 95.25 69.85) (xy 99.06 69.85))
-    (stroke (width 0) (type default))
-  )
   (wire (pts (xy 50.8 85.09) (xy 49.53 85.09))
     (stroke (width 0) (type default))
   )
-  (wire (pts (xy 95.25 64.77) (xy 114.3 64.77))
-    (stroke (width 0) (type default))
-  )
   (wire (pts (xy 40.64 67.31) (xy 40.64 64.77))
     (stroke (width 0) (type default))
@@
     (stroke (width 0) (type default))
   )
-  (wire (pts (xy 127 53.34) (xy 127 55.88))
+  (wire (pts (xy 127 50.8) (xy 127 52.07))
     (stroke (width 0) (type default))
   )
@@
     (stroke (width 0) (type default))
   )
+  (wire (pts (xy 63.5 36.83) (xy 68.58 36.83))
+    (stroke (width 0) (type default))
+  )
   (wire (pts (xy 80.01 99.06) (xy 85.09 99.06))
     (stroke (width 0) (type default))
   )
-  (wire (pts (xy 110.49 106.68) (xy 80.01 106.68))
-    (stroke (width 0) (type default))
-  )
   (wire (pts (xy 104.14 36.83) (xy 104.14 40.64))
     (stroke (width 0) (type default))
   )
-  (label "IR_sensor" (at 44.45 72.39 0) (fields_autoplaced)
+  (text "Изготвено от:\nA4 само хартия" (at 100.33 123.19 0)
+    (effects (font (size 3 3)) (justify left bottom))
+  )
+  (label "SDA" (at 80.01 104.14 0) (fields_autoplaced)
     (effects (font (size 1.27 1.27)) (justify left bottom))
   )
-  (label "IR_sensor" (at 99.06 69.85 0) (fields_autoplaced)
+  (label "SCL" (at 63.5 29.21 0) (fields_autoplaced)
     (effects (font (size 1.27 1.27)) (justify left bottom))
   )
+  (label "IR" (at 44.45 72.39 0) (fields_autoplaced)
+    (effects (font (size 1.27 1.27)) (justify left bottom))
+  )
+  (label "IR" (at 63.5 36.83 0) (fields_autoplaced)
+    (effects (font (size 1.27 1.27)) (justify left bottom))
+  )
+  (label "Motor" (at 63.5 34.29 0) (fields_autoplaced)
+    (effects (font (size 1.27 1.27)) (justify left bottom))
+  )
+  (label "Motor" (at 97.79 39.37 0) (fields_autoplaced)
+    (effects (font (size 1.27 1.27)) (justify left bottom))
+  )
+  (label "SDA" (at 63.5 31.75 0) (fields_autoplaced)
+    (effects (font (size 1.27 1.27)) (justify left bottom))
+  )
+  (label "SCL" (at 80.01 106.68 0) (fields_autoplaced)
+    (effects (font (size 1.27 1.27)) (justify left bottom))
+  )
   (symbol (lib_id "power:+3V3") (at 53.34 19.05 0) (unit 1)
     (in_bom yes) (on_board yes) (dnp no)
@@
     )
   )
-  (symbol (lib_id "power:GND") (at 64.77 34.29 0) (unit 1)
-    (in_bom yes) (on_board yes) (dnp no)
-    (property "Reference" "#PWR01" (at 64.77 40.64 0)
-      (effects (font (size 1.27 1.27)) hide)
-    )
-    (property "Value" "GND" (at 64.77 38.1 0)
-      (effects (font (size 1.27 1.27)))
-    )
-    (property "Footprint" "" (at 64.77 34.29 0)
-      (effects (font (size 1.27 1.27)) hide)
-    )
-    (property "Datasheet" "" (at 64.77 34.29 0)
-      (effects (font (size 1.27 1.27)) hide)
-    )
-    (pin "1")
-    (instances
-      (project "First_schemes"
-        (path "/e2e3fdbe-1c24-44db-9a9f-1c2ab1af1745"
-          (reference "#PWR01") (unit 1)
-        )
-      )
-    )
-  )
   (symbol (lib_id "power:+3V3") (at 40.64 25.4 0) (unit 1)
     (in_bom yes) (on_board yes) (dnp no)
@@
         (path "/e2e3fdbe-1c24-44db-9a9f-1c2ab1af1745"
           (reference "#PWR06") (unit 1)
+        )
+      )
+    )
+  )
+  (symbol (lib_id "power:+5V") (at 125.73 31.75 0) (unit 1)
+    (in_bom yes) (on_board yes) (dnp no)
+    (property "Reference" "#PWR012" (at 125.73 35.56 0)
+      (effects (font (size 1.27 1.27)) hide)
+    )
+    (property "Value" "+5V" (at 125.73 27.94 0)
+      (effects (font (size 1.27 1.27)))
+    )
+    (property "Footprint" "" (at 125.73 31.75 0)
+      (effects (font (size 1.27 1.27)) hide)
+    )
+    (property "Datasheet" "" (at 125.73 31.75 0)
+      (effects (font (size 1.27 1.27)) hide)
+    )
+    (pin "1")
+    (instances
+      (project "First_schemes"
+        (path "/e2e3fdbe-1c24-44db-9a9f-1c2ab1af1745"
+          (reference "#PWR012") (unit 1)
         )
       )
@@
     )
   )
-  (symbol (lib_id "power:GND") (at 127 55.88 0) (unit 1)
-    (in_bom yes) (on_board yes) (dnp no)
-    (property "Reference" "#PWR011" (at 127 62.23 0)
-      (effects (font (size 1.27 1.27)) hide)
-    )
-    (property "Value" "GND" (at 127 59.69 0)
-      (effects (font (size 1.27 1.27)))
-    )
-    (property "Footprint" "" (at 127 55.88 0)
-      (effects (font (size 1.27 1.27)) hide)
-    )
-    (property "Datasheet" "" (at 127 55.88 0)
+  (symbol (lib_id "power:GND") (at 127 52.07 0) (unit 1)
+    (in_bom yes) (on_board yes) (dnp no)
+    (property "Reference" "#PWR011" (at 127 58.42 0)
+      (effects (font (size 1.27 1.27)) hide)
+    )
+    (property "Value" "GND" (at 127 55.88 0)
+      (effects (font (size 1.27 1.27)))
+    )
+    (property "Footprint" "" (at 127 52.07 0)
+      (effects (font (size 1.27 1.27)) hide)
+    )
+    (property "Datasheet" "" (at 127 52.07 0)
       (effects (font (size 1.27 1.27)) hide)
     )
@@
     )
   )
-  (symbol (lib_id "Motor:Motor_DC") (at 127 45.72 0) (unit 1)
+  (symbol (lib_id "Motor:Motor_DC") (at 127 43.18 0) (unit 1)
     (in_bom yes) (on_board yes) (dnp no) (fields_autoplaced)
-    (property "Reference" "M1" (at 132.08 46.99 0)
+    (property "Reference" "M1" (at 132.08 44.45 0)
       (effects (font (size 1.27 1.27)) (justify left))
     )
-    (property "Value" "Motor" (at 132.08 49.53 0)
+    (property "Value" "Motor" (at 132.08 46.99 0)
       (effects (font (size 1.27 1.27)) (justify left))
     )
-    (property "Footprint" "" (at 127 48.006 0)
-      (effects (font (size 1.27 1.27)) hide)
-    )
-    (property "Datasheet" "~" (at 127 48.006 0)
+    (property "Footprint" "" (at 127 45.466 0)
+      (effects (font (size 1.27 1.27)) hide)
+    )
+    (property "Datasheet" "~" (at 127 45.466 0)
       (effects (font (size 1.27 1.27)) hide)
     )
@@
         )
       )
+    )
+  )
+  (symbol (lib_id "power:GND") (at 57.15 30.48 0) (unit 1)
+    (in_bom yes) (on_board yes) (dnp no)
+    (property "Reference" "#PWR01" (at 57.15 36.83 0)
+      (effects (font (size 1.27 1.27)) hide)
+    )
+    (property "Value" "GND" (at 57.15 34.29 0)
+      (effects (font (size 1.27 1.27)))
+    )
+    (property "Footprint" "" (at 57.15 30.48 0)
+      (effects (font (size 1.27 1.27)) hide)
+    )
+    (property "Datasheet" "" (at 57.15 30.48 0)
+      (effects (font (size 1.27 1.27)) hide)
+    )
+    (pin "1")
+    (instances
+      (project "First_schemes"
+        (path "/e2e3fdbe-1c24-44db-9a9f-1c2ab1af1745"
+          (reference "#PWR01") (unit 1)
+        )
+      )
